File: SingleActiveMarkerDeck.kicad_sch (KiCad schematic)
At the start: 19 parts, among them P1 CF_EXP_LEFT, P2 CF_EXP_RIGHT, U1 BCR421UW6Q-7, U2 STBB1-APUR, U3 DS28E05R+T

Commit message: added PDF of schematic
Other:
- company: (none) -> DASC Lab, University of Michigan
- title: (none) -> Crazyflie Active Vicon LED Deck
Changed lines of the file:
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@@
 	(generator_version "9.0")
 	(paper "A4")
+	(title_block
+		(title "Crazyflie Active Vicon LED Deck")
+		(date "2025-08-07")
+		(rev "v1.0")
+		(company "DASC Lab, University of Michigan")
+	)
 	(text "C2761795"
 		(exclude_from_sim no)
